Commit message: fix(sim): hold real time and produce an accurate map of the house
Measured on a 16-core WSL2 laptop, scored against the true geometry in
worlds/house.sdf. Before: real-time factor 0.10-0.45, and 18-64% of occupied
map cells on a real obstacle. After: RTF 1.00 headless (0.8-1.0 with the GUI),
map 8.0 x 6.0 m against 8.1 x 6.1 m of real wall, 100% of occupied cells within
10 cm of a real obstacle and 91% of visible faces mapped, on three runs.

Speed. None of it was the hardware.
- The container has no GPU device, so Mesa falls back to llvmpipe and the
  Gazebo GUI and the gpu_lidar are rasterised on the CPU. sim.launch.py built
  gz_args itself, so passing gz_args:= to go headless was silently ignored;
  add headless:=true. Add compose.wsl-gpu.yaml to hand WSL2's GPU to Mesa's
  d3d12 driver (Gazebo CPU with the GUI ~480% -> ~280%).
- 1 ms physics published /clock at 1 kHz and woke every use_sim_time node on
  each tick. Step at 4 ms.
- Gazebo's JointStatePublisher has no rate limit and pushed /joint_states
  through the bridge at ~415 Hz. Use the joint_state_publisher node the real
  robot already uses.

Map quality.
- The centre of mass sat over the wheel axle with only a rear caster, and the
  caster sat 2.5 mm below the wheel contacts. The robot rode nose-down, up to
  9.4 degrees, tilted >2 degrees in 98% of samples, and the lidar 11 cm off the
  floor mapped the floor as walls. Move the COM between axle and caster and
  level the caster: pitch now 0.1 degrees. Documented for the real build.
- With the robot fixed, sensors, odometry and scan timing all checked out
  against ground truth, yet half the map was still bent. slam_toolbox's default
  8 m loop search window accepted a wrong closure on revisiting a room, every
  run. Disabling loop closure gave a perfect map, which isolated it; tighten
  the search to the odometry neighbourhood and demand stronger matches instead,
  so the real robot keeps loop closure for drift.

Nav2 re-verified on the new map with the new physics: cross-room goals reached
through the doorways, confirmed against Gazebo's true pose.

Co-Authored-By: Claude Opus 5.5 <noreply@anthropic.com>

File: urdf/casabot.urdf.xacro (robot description, xacro)
@@ -12,9 +12,17 @@
   <xacro:property name="base_mass"        value="1.6"/>
   <xacro:property name="wheel_mass"       value="0.05"/>
+  <!-- Centre of mass, measured from the axle (+x forward). It MUST sit between
+       the axle and the rear caster: with it on the axle nothing holds the nose
+       up, the robot tips forward onto its chassis when it brakes, and the
+       lidar - only ~11 cm off the floor - starts painting the floor as walls.
+       On the real robot, put the battery toward the caster. -->
+  <xacro:property name="com_x"            value="-0.04"/>
+  <xacro:property name="caster_radius"    value="${base_clearance/2 + 0.005}"/>
   <material name="grey"><color rgba="0.3 0.3 0.32 1"/></material>
   <material name="dark"><color rgba="0.1 0.1 0.1 1"/></material>
   <material name="red"><color rgba="0.7 0.1 0.1 1"/></material>
-  <xacro:macro name="box_inertia" params="m x y z">
+  <xacro:macro name="box_inertia" params="m x y z ox:=0">
     <inertial>
+      <origin xyz="${ox} 0 0"/>
       <mass value="${m}"/>
       <inertia ixx="${m*(y*y+z*z)/12}" iyy="${m*(x*x+z*z)/12}" izz="${m*(x*x+y*y)/12}"
@@ -32,5 +40,5 @@
       <geometry><box size="${base_length} ${base_width} ${base_height}"/></geometry>
     </collision>
-    <xacro:box_inertia m="${base_mass}" x="${base_length}" y="${base_width}" z="${base_height}"/>
+    <xacro:box_inertia m="${base_mass}" x="${base_length}" y="${base_width}" z="${base_height}" ox="${com_x}"/>
   </link>
   <joint name="base_footprint_joint" type="fixed">
@@ -69,6 +77,6 @@
   <!-- Single rear ball caster. Modelled as a sphere so it slides in sim. -->
   <link name="caster_link">
-    <visual><geometry><sphere radius="${base_clearance/2 + 0.005}"/></geometry><material name="dark"/></visual>
-    <collision><geometry><sphere radius="${base_clearance/2 + 0.005}"/></geometry></collision>
+    <visual><geometry><sphere radius="${caster_radius}"/></geometry><material name="dark"/></visual>
+    <collision><geometry><sphere radius="${caster_radius}"/></geometry></collision>
     <inertial><mass value="0.02"/><inertia ixx="1e-5" iyy="1e-5" izz="1e-5" ixy="0" ixz="0" iyz="0"/></inertial>
   </link>
@@ -76,5 +84,7 @@
     <parent link="base_link"/>
     <child link="caster_link"/>
-    <origin xyz="${-base_length/2 + 0.03} 0 ${-base_height/2 - base_clearance/2 + 0.005}"/>
+    <!-- Bottom of the sphere exactly on the floor, level with the wheel
+         contacts. Any offset here is a permanent tilt of the lidar. -->
+    <origin xyz="${-base_length/2 + 0.03} 0 ${caster_radius - wheel_radius - base_clearance}"/>
   </joint>
   <link name="lidar_link">

File: urdf/gazebo.xacro (robot description, xacro)
@@ -20,8 +20,4 @@
       <child_frame_id>base_footprint</child_frame_id>
       <odom_publish_frequency>30</odom_publish_frequency>
-    </plugin>
-    <plugin filename="gz-sim-joint-state-publisher-system"
-            name="gz::sim::systems::JointStatePublisher">
-      <topic>joint_states</topic>
     </plugin>
   </gazebo>
